Commit message: Added joint 0, end effector; updated moveit_config

File: src/moveit_config/config/my_robot.ros2_control.xacro (robot description, xacro)
@@ -3,25 +3,59 @@
     <xacro:macro name="my_robot_ros2_control" params="name initial_positions_file">
         <xacro:property name="initial_positions" value="${xacro.load_yaml(initial_positions_file)['initial_positions']}"/>
-        <ros2_control name="RealHardware" type="system">
+        <ros2_control name="${name}" type="system">
             <hardware>
-                <plugin>canopen_ros2_control/Cia402System</plugin>
-                <param name="bus_config">$(find moveit_config)/config/bus.yml</param>
-                <param name="master_config">$(find moveit_config)/config/master.dcf</param>
-                <param name="can_interface_name">can0</param>
-                <param name="master_id">100</param>
-                <param name="config_fallback">true</param>
+                <!-- By default, set up controllers for simulation. This won't work on real hardware -->
+                <plugin>mock_components/GenericSystem</plugin>
             </hardware>
-            <joint name="joint3">
-                <param name="node_id">1</param>
+            <joint name="joint0">
                 <command_interface name="position"/>
-                <state_interface name="position"/>
+                <state_interface name="position">
+                  <param name="initial_value">${initial_positions['joint0']}</param>
+                </state_interface>
                 <state_interface name="velocity"/>
             </joint>
             <joint name="joint1">
                 <command_interface name="position"/>
-                <state_interface name="position"/>
+                <state_interface name="position">
+                  <param name="initial_value">${initial_positions['joint1']}</param>
+                </state_interface>
                 <state_interface name="velocity"/>
             </joint>
-    </ros2_control>
+            <joint name="joint2">
+                <command_interface name="position"/>
+                <state_interface name="position">
+                  <param name="initial_value">${initial_positions['joint2']}</param>
+                </state_interface>
+                <state_interface name="velocity"/>
+            </joint>
+            <joint name="joint3">
+                <command_interface name="position"/>
+                <state_interface name="position">
+                  <param name="initial_value">${initial_positions['joint3']}</param>
+                </state_interface>
+                <state_interface name="velocity"/>
+            </joint>
+            <joint name="joint4">
+                <command_interface name="position"/>
+                <state_interface name="position">
+                  <param name="initial_value">${initial_positions['joint4']}</param>
+                </state_interface>
+                <state_interface name="velocity"/>
+            </joint>
+            <joint name="joint5">
+                <command_interface name="position"/>
+                <state_interface name="position">
+                  <param name="initial_value">${initial_positions['joint5']}</param>
+                </state_interface>
+                <state_interface name="velocity"/>
+            </joint>
+            <joint name="joint6">
+                <command_interface name="position"/>
+                <state_interface name="position">
+                  <param name="initial_value">${initial_positions['joint6']}</param>
+                </state_interface>
+                <state_interface name="velocity"/>
+            </joint>
+        </ros2_control>
     </xacro:macro>
 </robot>

File: src/my_robot_description/urdf/arm.urdf.xacro (robot description, xacro)
@@ -3,3 +3,4 @@
     <xacro:include filename="common_properties.xacro"/>
     <xacro:include filename="arm.xacro"/>
+    <xacro:include filename="my_robot.ros2_control.xacro"/>
 </robot>

File: src/my_robot_description/urdf/arm.xacro (robot description, xacro)
@@ -2,4 +2,20 @@
 <robot xmlns:xacro="http://www.ros.org/wiki/xacro">
     <!-- Robot links -->
+    <link name="world_frame"/>  <!-- World frame link (reference frame for the robot) -->
+    <link name="linear_rail_link">
+        <visual>
+            <geometry>
+                <box size="2.9464 0.445 0.1016"/>  <!-- Visual geometry for the linear rail (box shape) -->
+            </geometry>
+            <origin xyz="0 0 0" rpy="0 0 0"/>       <!-- Origin of the visual element (centered on the linear rail) -->
+            <material name="grey"/>
+        </visual>
+        <collision>
+            <geometry>
+                <box size="2.9464 0.445 0.1016"/>  <!-- Collision geometry for the linear rail (box shape) -->
+            </geometry>
+            <origin xyz="0 0 0" rpy="0 0 0"/>       <!-- Origin of the collision element (centered on the linear rail) -->
+        </collision>
+    </link>
     <link name="base_link">
         <visual>
@@ -92,61 +108,74 @@
         </collision>
     </link>
+    <!-- End-effector (box of approximate size for now) -->
     <link name="link6">
         <visual>
             <geometry>
-                <box size="0.05 0.05 0.05"/>
+                <box size="0.12 0.12 0.26"/>
             </geometry>
-            <origin xyz="0 0 0.025" rpy="0 0 0"/>
+            <origin xyz="0 0 0.13" rpy="0 0 0"/>
             <material name="grey"/>
         </visual>
         <collision>
             <geometry>
-                <box size="0.05 0.05 0.05"/>
+                <box size="0.12 0.12 0.26"/>
             </geometry>
-            <origin xyz="0 0 0.025" rpy="0 0 0"/>
+            <origin xyz="0 0 0.13" rpy="0 0 0"/>
         </collision>
     </link>
     <!-- Robot joints -->
+    <joint name="world_to_linear_rail" type="fixed">
+        <parent link="world_frame"/>                                            <!-- Parent link for the fixed joint (world frame) -->
+        <child link="linear_rail_link"/>                                        <!-- Child link for the fixed joint (linear rail) -->
+        <origin xyz="0 0 0" rpy="0 0 0"/>                                       <!-- Origin of the joint (position and orientation of the linear rail in the world frame) -->
+    </joint>
+    <joint name="joint0" type="prismatic">
+        <parent link="linear_rail_link"/>                                       <!-- Parent link for joint0 -->
+        <child link="base_link"/>                                               <!-- Child link for joint0 -->
+        <origin xyz="0 0 0.0508" rpy="0 0 0"/>                                  <!-- Origin of the joint -->
+        <axis xyz="1 0 0"/>                                                     <!-- Axis of translation for the prismatic joint (x-axis) -->
+        <limit effort="100" velocity="0.5" lower="-0.85" upper="0.85"/>         <!-- Joint limits (effort, velocity, lower and upper translation limits in meters) !! CHANGE LATER !! -->
+    </joint>
     <joint name="joint1" type="revolute">
-        <parent link="base_link"/>                                          <!-- Parent link for joint1 -->
-        <child link="link1"/>                                               <!-- Child link for joint1 -->
-        <origin xyz="0 0 0" rpy="0 0 0"/>                                   <!-- Origin of the joint -->
-        <axis xyz="0 0 1"/>                                                 <!-- Axis of rotation for the revolute joint (z-axis) -->
-        <limit effort="37" velocity="0.4" lower="-3.14" upper="3.14"/>  <!-- Joint limits (effort, velocity, lower and upper angle limits in radians) -->
+        <parent link="base_link"/>                                              <!-- Parent link for joint1 -->
+        <child link="link1"/>                                                   <!-- Child link for joint1 -->
+        <origin xyz="0 0 0" rpy="0 0 0"/>                                       <!-- Origin of the joint -->
+        <axis xyz="0 0 1"/>                                                     <!-- Axis of rotation for the revolute joint (z-axis) -->
+        <limit effort="37" velocity="0.4" lower="-3.14" upper="3.14"/>          <!-- Joint limits (effort, velocity, lower and upper angle limits in radians) -->
     </joint>
     <joint name="joint2" type="revolute">
-        <parent link="link1"/>                                              <!-- Parent link for joint2 -->
-        <child link="link2"/>                                               <!-- Child link for joint2 -->
-        <origin xyz="-0.145 0 0.212599" rpy="0 0 0"/>                       <!-- Origin of the joint -->
-        <axis xyz="1 0 0"/>                                                 <!-- Axis of rotation for the revolute joint (z-axis) -->
+        <parent link="link1"/>                                                  <!-- Parent link for joint2 -->
+        <child link="link2"/>                                                   <!-- Child link for joint2 -->
+        <origin xyz="-0.145 0 0.212599" rpy="0 0 0"/>                           <!-- Origin of the joint -->
+        <axis xyz="1 0 0"/>                                                     <!-- Axis of rotation for the revolute joint (z-axis) -->
         <limit effort="144" velocity="1.96" lower="-1.57079" upper="1.57079"/>  <!-- Joint limits (effort, velocity, lower and upper angle limits in radians) -->
     </joint>
     <joint name="joint3" type="revolute">
-        <parent link="link2"/>                                              <!-- Parent link for joint3 -->
-        <child link="link3"/>                                               <!-- Child link for joint3 -->
+        <parent link="link2"/>                                                  <!-- Parent link for joint3 -->
+        <child link="link3"/>                                                   <!-- Child link for joint3 -->
         <origin xyz="-0.017125 0 0.663309" rpy="0 -1.57079 3.14195"/>                                   <!-- Origin of the joint -->
-        <axis xyz="0 0 1"/>                                                 <!-- Axis of rotation for the revolute joint (z-axis) -->
-        <limit effort="77" velocity="3.65" lower="-4.5" upper="1.4"/>  <!-- Joint limits (effort, velocity, lower and upper angle limits in radians) -->
+        <axis xyz="0 0 1"/>                                                     <!-- Axis of rotation for the revolute joint (z-axis) -->
+        <limit effort="77" velocity="3.65" lower="-4.5" upper="1.4"/>           <!-- Joint limits (effort, velocity, lower and upper angle limits in radians) -->
     </joint>
     <joint name="joint4" type="revolute">
-        <parent link="link3"/>                                              <!-- Parent link for joint4 -->
-        <child link="link4"/>                                               <!-- Child link for joint4 -->
+        <parent link="link3"/>                                                  <!-- Parent link for joint4 -->
+        <child link="link4"/>                                                   <!-- Child link for joint4 -->
         <origin xyz="0 0.083285 0.08" rpy="-1.57079 0 0"/>                                   <!-- Origin of the joint -->
-        <axis xyz="0 0 1"/>                                                 <!-- Axis of rotation for the revolute joint (z-axis) -->
-        <limit effort="25" velocity="2" lower="-3.14159" upper="3.14159"/>  <!-- Joint limits (effort, velocity, lower and upper angle limits in radians) -->
+        <axis xyz="0 0 1"/>                                                     <!-- Axis of rotation for the revolute joint (z-axis) -->
+        <limit effort="25" velocity="2" lower="-3.14159" upper="3.14159"/>      <!-- Joint limits (effort, velocity, lower and upper angle limits in radians) -->
     </joint>
     <joint name="joint5" type="revolute">
-        <parent link="link4"/>                                              <!-- Parent link for joint5 -->
-        <child link="link5"/>                                               <!-- Child link for joint5 -->
-        <origin xyz="-0.054 0 0.4645" rpy="0 1.57079 0"/>                                   <!-- Origin of the joint -->
-        <axis xyz="0 0 1"/>                                                 <!-- Axis of rotation for the revolute joint (z-axis) -->
-        <limit effort="24" velocity="3.5" lower="-3.14159" upper="3.14159"/>  <!-- Joint limits (effort, velocity, lower and upper angle limits in radians) -->
+        <parent link="link4"/>                                                  <!-- Parent link for joint5 -->
+        <child link="link5"/>                                                   <!-- Child link for joint5 -->
+        <origin xyz="-0.054 0 0.4645" rpy="0 1.57079 0"/>                       <!-- Origin of the joint -->
+        <axis xyz="0 0 1"/>                                                     <!-- Axis of rotation for the revolute joint (z-axis) -->
+        <limit effort="24" velocity="3.5" lower="-3.14159" upper="3.14159"/>    <!-- Joint limits (effort, velocity, lower and upper angle limits in radians) -->
     </joint>
     <joint name="joint6" type="revolute">
-        <parent link="link5"/>                                              <!-- Parent link for joint6 -->
-        <child link="link6"/>                                               <!-- Child link for joint6 -->
-        <origin xyz="-0.047 0 -0.055033" rpy="0 -1.57079 0"/>               <!-- Origin of the joint -->
-        <axis xyz="0 0 1"/>                                                 <!-- Axis of rotation for the revolute joint (z-axis) -->
-        <limit effort="12" velocity="3.5" lower="-1.57079" upper="1.57079"/>  <!-- Joint limits (effort, velocity, lower and upper angle limits in radians) -->
+        <parent link="link5"/>                                                  <!-- Parent link for joint6 -->
+        <child link="link6"/>                                                   <!-- Child link for joint6 -->
+        <origin xyz="-0.047 0 -0.055033" rpy="0 -1.57079 0"/>                   <!-- Origin of the joint -->
+        <axis xyz="0 0 1"/>                                                     <!-- Axis of rotation for the revolute joint (z-axis) -->
+        <limit effort="12" velocity="3.5" lower="-1.57079" upper="1.57079"/>    <!-- Joint limits (effort, velocity, lower and upper angle limits in radians) -->
     </joint>
 </robot>
