Commit message: build(URDF): :wrench: Add gripper to MoveIt config
Add gripper to MoveIt configuration files

Co-authored-by: Copilot <copilot@github.com>

File: src/moveit_config/config/robot.ros2_control.xacro (robot description, xacro)
@@ -5,5 +5,5 @@
             <hardware>
                 <!-- By default, set up controllers for simulation. This won't work on real hardware -->
-            <plugin>mock_components/GenericSystem</plugin>
+                <plugin>mock_components/GenericSystem</plugin>
             </hardware>
             <joint name="joint0">
@@ -49,5 +49,6 @@
                 <state_interface name="velocity"/>
             </joint>
-            <joint name="joint6">
+            <!-- Gripper: only finger_1 needs a command interface; fingers 2 & 3 are mimic -->
+            <joint name="finger_1_joint">
                 <command_interface name="position"/>
                 <state_interface name="position">

Commit message: fix(URDF): :wrench: Fix config files for addition of gripper
Fix description, bringup, and moveit config files for addition of the gripper

Co-authored-by: Copilot <copilot@github.com>

File: src/moveit_config/config/robot.ros2_control.xacro (robot description, xacro)
@@ -49,5 +49,5 @@
                 <state_interface name="velocity"/>
             </joint>
-            <!-- Gripper: only finger_1 needs a command interface; fingers 2 & 3 are mimic -->
+            <!-- Gripper - only finger_1 needs a command interface; fingers 2 & 3 are mimic -->
             <joint name="finger_1_joint">
                 <command_interface name="position"/>

File: src/robot_description/urdf/robot.ros2_control.xacro (robot description, xacro)
@@ -5,5 +5,5 @@
             <hardware>
                 <!-- By default, set up controllers for simulation. This won't work on real hardware -->
-            <plugin>mock_components/GenericSystem</plugin>
+                <plugin>mock_components/GenericSystem</plugin>
             </hardware>
             <joint name="joint0">
@@ -49,5 +49,6 @@
                 <state_interface name="velocity"/>
             </joint>
-            <joint name="gripper_joint">
+            <!-- Gripper - only finger_1 needs a command interface; fingers 2 & 3 are mimic -->
+            <joint name="finger_1_joint">
                 <command_interface name="position"/>
                 <state_interface name="position">
