Commit message: revert(MoveIt): :rewind: Revert addition of mock gripper
Revert addition of mock gripper

File: src/moveit_config/config/robot.ros2_control.xacro (robot description, xacro)
@@ -49,12 +49,4 @@
                 <state_interface name="velocity"/>
             </joint>
-            <!-- Gripper - only finger_1 needs a command interface; fingers 2 & 3 are mimic -->
-            <joint name="finger_1_joint">
-                <command_interface name="position"/>
-                <state_interface name="position">
-                    <param name="initial_value">0.0</param>
-                </state_interface>
-                <state_interface name="velocity"/>
-            </joint>
         </ros2_control>
     </xacro:macro>

File: src/robot_description/urdf/robot.ros2_control.xacro (robot description, xacro)
@@ -49,12 +49,4 @@
                 <state_interface name="velocity"/>
             </joint>
-            <!-- Gripper - only finger_1 needs a command interface; fingers 2 & 3 are mimic -->
-            <joint name="finger_1_joint">
-                <command_interface name="position"/>
-                <state_interface name="position">
-                    <param name="initial_value">0.0</param>
-                </state_interface>
-                <state_interface name="velocity"/>
-            </joint>
         </ros2_control>
     </xacro:macro>

File: src/robot_description/urdf/robot.urdf.xacro (robot description, xacro)
@@ -5,10 +5,3 @@
     <xacro:include filename="robot.ros2_control.xacro"/>
     <xacro:robot_ros2_control name="FakeSystem" initial_positions_file="unused"/>
-    <!-- Gripper -->
-    <xacro:include filename="gripper.xacro"/>
-    <joint name="gripper_mount" type="fixed">
-        <parent link="link5"/>
-        <child  link="gripper_base_link"/>
-        <origin xyz="-0.047 0 -0.055" rpy="3.14159 1.5708 0"/>
-    </joint>
 </robot>

File: src/robot_description/urdf/robot.xacro (robot description, xacro)
@@ -2,5 +2,4 @@
 <robot xmlns:xacro="http://www.ros.org/wiki/xacro">
     <!-- Robot links -->
-    <link name="world_frame"/>  <!-- World frame link (reference frame for the robot) -->
     <link name="linear_rail_link">
         <visual>

Commit message: fix(MoveIt): :bug: Fix URDF and MoveIt config bug after reverting previous commits

File: src/moveit_config/config/robot.ros2_control.xacro (robot description, xacro)
@@ -49,4 +49,11 @@
                 <state_interface name="velocity"/>
             </joint>
+            <joint name="joint6">
+                <command_interface name="position"/>
+                <state_interface name="position">
+                    <param name="initial_value">0.0</param>
+                </state_interface>
+                <state_interface name="velocity"/>
+            </joint>
         </ros2_control>
     </xacro:macro>

File: src/robot_description/urdf/robot.xacro (robot description, xacro)
@@ -2,4 +2,5 @@
 <robot xmlns:xacro="http://www.ros.org/wiki/xacro">
     <!-- Robot links -->
+    <link name="world_frame"/>  <!-- World frame link (no visual or collision geometry, serves as the root of the robot) -->
     <link name="linear_rail_link">
         <visual>

Commit message: feat(URDF): :wrench: Add gripper to configuration files
Add gripper to configuration files

File: src/moveit_config/config/robot.ros2_control.xacro (robot description, xacro)
@@ -49,5 +49,5 @@
                 <state_interface name="velocity"/>
             </joint>
-            <joint name="joint6">
+            <joint name="fin_joint1">
                 <command_interface name="position"/>
                 <state_interface name="position">

File: src/moveit_config/config/robot.urdf.xacro (robot description, xacro)
@@ -4,6 +4,3 @@
     <!-- Import robot urdf file -->
     <xacro:include filename="$(find robot_description)/urdf/robot.urdf.xacro" />
-    <!-- Import control_xacro -->
-    <xacro:include filename="robot.ros2_control.xacro" />
-    <xacro:robot_ros2_control name="FakeSystem" initial_positions_file="$(arg initial_positions_file)"/>
 </robot>

File: src/robot_description/urdf/robot.xacro (robot description, xacro)
@@ -6,12 +6,12 @@
         <visual>
             <geometry>
-                <box size="2.97 0.45 0.082"/>                                                                        <!-- Visual geometry for the linear rail (box shape) -->
-            </geometry>
-            <origin xyz="0 0 0" rpy="0 0 0"/>
-            <material name="grey"/>
-        </visual>
-        <collision>
-            <geometry>
-                <box size="2.97 0.45 0.082"/>                                                                        <!-- Collision geometry for the linear rail (box shape) -->
+                <box size="2.97 0.45 0.082"/>                                                                                <!-- Visual geometry for the linear rail (box shape) -->
+            </geometry>
+            <origin xyz="0 0 0" rpy="0 0 0"/>
+            <material name="grey"/>
+        </visual>
+        <collision>
+            <geometry>
+                <box size="2.97 0.45 0.082"/>                                                                                <!-- Collision geometry for the linear rail (box shape) -->
             </geometry>
             <origin xyz="0 0 0" rpy="0 0 0"/>
@@ -21,12 +21,12 @@
         <visual>
             <geometry>
-                <mesh filename="package://robot_description/meshes/Base Link Visual.stl" scale="0.001 0.001 0.001"/>     <!-- Visual geometry for the base link (STL file) -->
-            </geometry>
-            <origin xyz="0 0 0" rpy="0 0 0"/>
-            <material name="grey"/>
-        </visual>
-        <collision>
-            <geometry>
-                <mesh filename="package://robot_description/meshes/Base Link Collision.stl" scale="0.001 0.001 0.001"/>  <!-- Collision geometry for the base link (STL file) -->
+                <mesh filename="package://robot_description/meshes/Base Link Visual.stl" scale="0.001 0.001 0.001"/>         <!-- Visual geometry for the base link (STL file) -->
+            </geometry>
+            <origin xyz="0 0 0" rpy="0 0 0"/>
+            <material name="grey"/>
+        </visual>
+        <collision>
+            <geometry>
+                <mesh filename="package://robot_description/meshes/Base Link Collision.stl" scale="0.001 0.001 0.001"/>      <!-- Collision geometry for the base link (STL file) -->
             </geometry>
             <origin xyz="0 0 0" rpy="0 0 0"/>
@@ -36,5 +36,5 @@
         <visual>
             <geometry>
-                <mesh filename="package://robot_description/meshes/Link 1 Visual.stl" scale="0.001 0.001 0.001"/>        <!-- Visual geometry for the link 1 (STL file) -->
+                <mesh filename="package://robot_description/meshes/Link 1 Visual.stl" scale="0.001 0.001 0.001"/>            <!-- Visual geometry for the link 1 (STL file) -->
             </geometry>
             <origin xyz="0 0 0" rpy="0 0 0"/>
@@ -43,5 +43,5 @@
         <collision>
             <geometry>
-                <mesh filename="package://robot_description/meshes/Link 1 Collision.stl" scale="0.001 0.001 0.001"/>     <!-- Collision geometry for the link 1 (STL file) -->
+                <mesh filename="package://robot_description/meshes/Link 1 Collision.stl" scale="0.001 0.001 0.001"/>         <!-- Collision geometry for the link 1 (STL file) -->
             </geometry>
             <origin xyz="0 0 0" rpy="0 0 0"/>
@@ -51,5 +51,5 @@
         <visual>
             <geometry>
-                <mesh filename="package://robot_description/meshes/Link 2 Visual.stl" scale="0.001 0.001 0.001"/>        <!-- Visual geometry for the link 2 (STL file) -->
+                <mesh filename="package://robot_description/meshes/Link 2 Visual.stl" scale="0.001 0.001 0.001"/>            <!-- Visual geometry for the link 2 (STL file) -->
             </geometry>
             <origin xyz="0 0 0" rpy="0 0 0"/>
@@ -58,5 +58,5 @@
         <collision>
             <geometry>
-                <mesh filename="package://robot_description/meshes/Link 2 Collision.stl" scale="0.001 0.001 0.001"/>     <!-- Collision geometry for the link 2 (STL file) -->
+                <mesh filename="package://robot_description/meshes/Link 2 Collision.stl" scale="0.001 0.001 0.001"/>         <!-- Collision geometry for the link 2 (STL file) -->
             </geometry>
             <origin xyz="0 0 0" rpy="0 0 0"/>
@@ -66,5 +66,5 @@
         <visual>
             <geometry>
-                <mesh filename="package://robot_description/meshes/Link 3 Visual.stl" scale="0.001 0.001 0.001"/>        <!-- Visual geometry for the link 3 (STL file) -->
+                <mesh filename="package://robot_description/meshes/Link 3 Visual.stl" scale="0.001 0.001 0.001"/>            <!-- Visual geometry for the link 3 (STL file) -->
             </geometry>
             <origin xyz="0 0 0" rpy="0 0 0"/>
@@ -73,5 +73,5 @@
         <collision>
             <geometry>
-                <mesh filename="package://robot_description/meshes/Link 3 Collision.stl" scale="0.001 0.001 0.001"/>     <!-- Collision geometry for the link 3 (STL file) -->
+                <mesh filename="package://robot_description/meshes/Link 3 Collision.stl" scale="0.001 0.001 0.001"/>         <!-- Collision geometry for the link 3 (STL file) -->
             </geometry>
             <origin xyz="0 0 0" rpy="0 0 0"/>
@@ -81,5 +81,5 @@
         <visual>
             <geometry>
-                <mesh filename="package://robot_description/meshes/Link 4 Visual.stl" scale="0.001 0.001 0.001"/>       <!-- Visual geometry for the link 4 (STL file) -->
+                <mesh filename="package://robot_description/meshes/Link 4 Visual.stl" scale="0.001 0.001 0.001"/>            <!-- Visual geometry for the link 4 (STL file) -->
             </geometry>
             <origin xyz="0 0 0" rpy="0 0 0"/>
@@ -88,5 +88,5 @@
         <collision>
             <geometry>
-                <mesh filename="package://robot_description/meshes/Link 4 Collision.stl" scale="0.001 0.001 0.001"/>    <!-- Collision geometry for the link 4 (STL file) -->
+                <mesh filename="package://robot_description/meshes/Link 4 Collision.stl" scale="0.001 0.001 0.001"/>         <!-- Collision geometry for the link 4 (STL file) -->
             </geometry>
             <origin xyz="0 0 0" rpy="0 0 0"/>
@@ -96,5 +96,5 @@
         <visual>
             <geometry>
-                <mesh filename="package://robot_description/meshes/Link 5 Visual.stl" scale="0.001 0.001 0.001"/>       <!-- Visual geometry for the link 5 (STL file) -->
+                <mesh filename="package://robot_description/meshes/Link 5 Visual.stl" scale="0.001 0.001 0.001"/>            <!-- Visual geometry for the link 5 (STL file) -->
             </geometry>
             <origin xyz="0 0 0" rpy="0 0 0"/>
@@ -103,5 +103,5 @@
         <collision>
             <geometry>
-                <mesh filename="package://robot_description/meshes/Link 5 Collision.stl" scale="0.001 0.001 0.001"/>    <!-- Collision geometry for the link 5 (STL file) -->
+                <mesh filename="package://robot_description/meshes/Link 5 Collision.stl" scale="0.001 0.001 0.001"/>         <!-- Collision geometry for the link 5 (STL file) -->
             </geometry>
             <origin xyz="0 0 0" rpy="0 0 0"/>
@@ -111,5 +111,5 @@
         <visual>
             <geometry>
-                <mesh filename="package://robot_description/meshes/End Effector Geometry.stl" scale="0.001 0.001 0.001"/>       <!-- Visual geometry for the end-effector link (STL file) -->
+                <mesh filename="package://robot_description/meshes/End Effector Geometry.stl" scale="0.001 0.001 0.001"/>    <!-- Visual geometry for the end-effector link (STL file) -->
             </geometry>
             <origin xyz="0 0 0" rpy="0 0 0"/>
@@ -126,12 +126,12 @@
         <visual>
             <geometry>
-                <mesh filename="package://robot_description/meshes/Gripper fin.stl" scale="0.001 0.001 0.001"/>       <!-- Visual geometry for the fin link 1 (STL file) -->
-            </geometry>
-            <origin xyz="0 0 0" rpy="0 0 0"/>
-            <material name="grey"/>
-        </visual>
-        <collision>
-            <geometry>
-                <mesh filename="package://robot_description/meshes/Gripper fin.stl" scale="0.001 0.001 0.001"/>    <!-- Collision geometry for the fin link 1 (STL file) -->
+                <mesh filename="package://robot_description/meshes/Gripper fin.stl" scale="0.001 0.001 0.001"/>              <!-- Visual geometry for the fin link 1 (STL file) -->
+            </geometry>
+            <origin xyz="0 0 0" rpy="0 0 0"/>
+            <material name="grey"/>
+        </visual>
+        <collision>
+            <geometry>
+                <mesh filename="package://robot_description/meshes/Gripper fin.stl" scale="0.001 0.001 0.001"/>
             </geometry>
             <origin xyz="0 0 0" rpy="0 0 0"/>
@@ -141,12 +141,12 @@
         <visual>
             <geometry>
-                <mesh filename="package://robot_description/meshes/Gripper fin.stl" scale="0.001 0.001 0.001"/>       <!-- Visual geometry for the fin link 1 (STL file) -->
-            </geometry>
-            <origin xyz="0 0 0" rpy="0 0 0"/>
-            <material name="grey"/>
-        </visual>
-        <collision>
-            <geometry>
-                <mesh filename="package://robot_description/meshes/Gripper fin.stl" scale="0.001 0.001 0.001"/>    <!-- Collision geometry for the fin link 1 (STL file) -->
+                <mesh filename="package://robot_description/meshes/Gripper fin.stl" scale="0.001 0.001 0.001"/>              <!-- Visual geometry for the fin link 1 (STL file) -->
+            </geometry>
+            <origin xyz="0 0 0" rpy="0 0 0"/>
+            <material name="grey"/>
+        </visual>
+        <collision>
+            <geometry>
+                <mesh filename="package://robot_description/meshes/Gripper fin.stl" scale="0.001 0.001 0.001"/>
             </geometry>
             <origin xyz="0 0 0" rpy="0 0 0"/>
@@ -156,12 +156,12 @@
         <visual>
             <geometry>
-                <mesh filename="package://robot_description/meshes/Gripper fin.stl" scale="0.001 0.001 0.001"/>       <!-- Visual geometry for the fin link 1 (STL file) -->
-            </geometry>
-            <origin xyz="0 0 0" rpy="0 0 0"/>
-            <material name="grey"/>
-        </visual>
-        <collision>
-            <geometry>
-                <mesh filename="package://robot_description/meshes/Gripper fin.stl" scale="0.001 0.001 0.001"/>    <!-- Collision geometry for the fin link 1 (STL file) -->
+                <mesh filename="package://robot_description/meshes/Gripper fin.stl" scale="0.001 0.001 0.001"/>              <!-- Visual geometry for the fin link 1 (STL file) -->
+            </geometry>
+            <origin xyz="0 0 0" rpy="0 0 0"/>
+            <material name="grey"/>
+        </visual>
+        <collision>
+            <geometry>
+                <mesh filename="package://robot_description/meshes/Gripper fin.stl" scale="0.001 0.001 0.001"/>
             </geometry>
             <origin xyz="0 0 0" rpy="0 0 0"/>
@@ -198,5 +198,5 @@
         <parent link="link2"/>                                                  <!-- Parent link for joint3 -->
         <child link="link3"/>                                                   <!-- Child link for joint3 -->
-        <origin xyz="-0.017125 0 0.663309" rpy="0 -1.57079 3.14195"/>                                   <!-- Origin of the joint -->
+        <origin xyz="-0.017125 0 0.663309" rpy="0 -1.57079 3.14195"/>           <!-- Origin of the joint -->
         <axis xyz="0 0 1"/>                                                     <!-- Axis of rotation for the revolute joint (z-axis) -->
         <limit effort="77" velocity="3.65" lower="-4.5" upper="1.4"/>           <!-- Joint limits (effort, velocity, lower and upper angle limits in radians) -->
@@ -205,5 +205,5 @@
         <parent link="link3"/>                                                  <!-- Parent link for joint4 -->
         <child link="link4"/>                                                   <!-- Child link for joint4 -->
-        <origin xyz="0 0.083285 0.08" rpy="-1.57079 0 0"/>                                   <!-- Origin of the joint -->
+        <origin xyz="0 0.083285 0.08" rpy="-1.57079 0 0"/>                      <!-- Origin of the joint -->
         <axis xyz="0 0 1"/>                                                     <!-- Axis of rotation for the revolute joint (z-axis) -->
         <limit effort="25" velocity="2" lower="-3.14159" upper="3.14159"/>      <!-- Joint limits (effort, velocity, lower and upper angle limits in radians) -->
@@ -225,14 +225,14 @@
         <parent link="link6"/>                                                  <!-- Parent link for fin_joint1 -->
         <child link="fin_link1"/>                                               <!-- Child link for fin_joint1 -->
-        <origin xyz="0.049999999 0 0.1355" rpy="0 0 3.14159"/>                  <!-- Origin of the joint -->
+        <origin xyz="0.05052 0 0.1355" rpy="0 0 3.14159"/>                      <!-- Origin of the joint (hinge hole center at r=50.52mm, z=135.5mm) -->
         <axis xyz="0 1 0"/>                                                     <!-- Axis of rotation for the revolute joint (y-axis) -->
-        <limit effort="10" velocity="1.0" lower="-1.0" upper="1.0"/>               <!-- Joint limits (effort, velocity, lower and upper angle limits in radians) -->
+        <limit effort="10" velocity="1.0" lower="-0.25" upper="0.175"/>            <!-- Joint limits (effort, velocity, lower and upper angle limits in radians) -->
     </joint>
     <joint name="fin_joint2" type="revolute">
         <parent link="link6"/>                                                  <!-- Parent link for fin_joint2 -->
         <child link="fin_link2"/>                                               <!-- Child link for fin_joint2 -->
-        <origin xyz="-0.025 0.0433 0.1255" rpy="0 0 5.23599"/>                        <!-- Origin of the joint -->
+        <origin xyz="-0.02526 0.04375 0.1355" rpy="0 0 5.23599"/>               <!-- Origin of the joint (hinge hole center at r=50.52mm, 120°, z=135.5mm) -->
         <axis xyz="0 1 0"/>                                                     <!-- Axis of rotation for the revolute joint (y-axis) -->
-        <limit effort="10" velocity="1.0" lower="-1.0" upper="1.0"/>               <!-- Joint limits (effort, velocity, lower and upper angle limits in radians) -->
+        <limit effort="10" velocity="1.0" lower="-1.0" upper="1.0"/>            <!-- Joint limits (effort, velocity, lower and upper angle limits in radians) -->
         <mimic joint="fin_joint1" multiplier="1.0" offset="0.0"/>               <!-- Mimic joint definition to mirror the motion of fin_joint1 -->
     </joint>
@@ -240,7 +240,7 @@
         <parent link="link6"/>                                                  <!-- Parent link for fin_joint3 -->
         <child link="fin_link3"/>                                               <!-- Child link for fin_joint3 -->
-        <origin xyz="-0.025 -0.0433 0.1255" rpy="0 0 7.33039"/>                       <!-- Origin of the joint -->
+        <origin xyz="-0.02526 -0.04375 0.1355" rpy="0 0 7.33039"/>              <!-- Origin of the joint (hinge hole center at r=50.52mm, 240°, z=135.5mm) -->
         <axis xyz="0 1 0"/>                                                     <!-- Axis of rotation for the revolute joint (y-axis) -->
-        <limit effort="10" velocity="1.0" lower="-1.0" upper="1.0"/>               <!-- Joint limits (effort, velocity, lower and upper angle limits in radians) -->
+        <limit effort="10" velocity="1.0" lower="-1.0" upper="1.0"/>            <!-- Joint limits (effort, velocity, lower and upper angle limits in radians) -->
         <mimic joint="fin_joint1" multiplier="1.0" offset="0.0"/>               <!-- Mimic joint definition to mirror the motion of fin_joint1 -->
     </joint>

Commit message: build(MoveIt): :wrench: Update joint 6 to be revolute
Update joint 6 to be revolute instead of fixed

File: src/moveit_config/config/robot.ros2_control.xacro (robot description, xacro)
@@ -49,4 +49,11 @@
                 <state_interface name="velocity"/>
             </joint>
+            <joint name="joint6">
+                <command_interface name="position"/>
+                <state_interface name="position">
+                    <param name="initial_value">0.0</param>
+                </state_interface>
+                <state_interface name="velocity"/>
+            </joint>
             <joint name="fin_joint1">
                 <command_interface name="position"/>
