Commit message: feat(URDF): :sparkles: Add mock gripper to robot model
Add mock gripper to robot URDF

Co-authored-by: Copilot <copilot@github.com>

File: src/robot_description/urdf/robot.ros2_control.xacro (robot description, xacro)
@@ -49,5 +49,5 @@
                 <state_interface name="velocity"/>
             </joint>
-            <joint name="joint6">
+            <joint name="gripper_joint">
                 <command_interface name="position"/>
                 <state_interface name="position">

File: src/robot_description/urdf/robot.urdf.xacro (robot description, xacro)
@@ -5,3 +5,10 @@
     <xacro:include filename="robot.ros2_control.xacro"/>
     <xacro:robot_ros2_control name="FakeSystem" initial_positions_file="unused"/>
+    <!-- Gripper -->
+    <xacro:include filename="gripper.xacro"/>
+    <joint name="gripper_mount" type="fixed">
+        <parent link="link5"/>
+        <child  link="gripper_base_link"/>
+        <origin xyz="-0.047 0 -0.055" rpy="3.14159 1.5708 0"/>
+    </joint>
 </robot>

File: src/robot_description/urdf/robot.xacro (robot description, xacro)
@@ -108,20 +108,4 @@
         </collision>
     </link>
-    <!-- End-effector (box of approximate size for now) -->
-    <link name="link6">
-        <visual>
-            <geometry>
-                <box size="0.12 0.12 0.26"/>
-            </geometry>
-            <origin xyz="0 0 0.13" rpy="0 0 0"/>
-            <material name="grey"/>
-        </visual>
-        <collision>
-            <geometry>
-                <box size="0.12 0.12 0.26"/>
-            </geometry>
-            <origin xyz="0 0 0.13" rpy="0 0 0"/>
-        </collision>
-    </link>
     <!-- Robot joints -->
     <joint name="world_to_linear_rail" type="fixed">
@@ -172,10 +156,3 @@
         <limit effort="24" velocity="3.5" lower="-3.14159" upper="3.14159"/>    <!-- Joint limits (effort, velocity, lower and upper angle limits in radians) -->
     </joint>
-    <joint name="joint6" type="revolute">
-        <parent link="link5"/>                                                  <!-- Parent link for joint6 -->
-        <child link="link6"/>                                                   <!-- Child link for joint6 -->
-        <origin xyz="-0.047 0 -0.055033" rpy="0 -1.57079 0"/>                   <!-- Origin of the joint -->
-        <axis xyz="0 0 1"/>                                                     <!-- Axis of rotation for the revolute joint (z-axis) -->
-        <limit effort="12" velocity="3.5" lower="-1.57079" upper="1.57079"/>    <!-- Joint limits (effort, velocity, lower and upper angle limits in radians) -->
-    </joint>
 </robot>
