Commit message: revert(URDF): :rewind: Revert "feat(URDF): :sparkles: Add mock gripper to robot model"
This reverts commit 15d5415c9ed845268dcb3cd48c87c456982c850f.

File: src/robot_description/urdf/robot.ros2_control.xacro (robot description, xacro)
@@ -5,5 +5,5 @@
             <hardware>
                 <!-- By default, set up controllers for simulation. This won't work on real hardware -->
-                <plugin>mock_components/GenericSystem</plugin>
+            <plugin>mock_components/GenericSystem</plugin>
             </hardware>
             <joint name="joint0">
@@ -49,4 +49,11 @@
                 <state_interface name="velocity"/>
             </joint>
+            <joint name="joint6">
+                <command_interface name="position"/>
+                <state_interface name="position">
+                    <param name="initial_value">0.0</param>
+                </state_interface>
+                <state_interface name="velocity"/>
+            </joint>
         </ros2_control>
     </xacro:macro>

File: src/robot_description/urdf/robot.xacro (robot description, xacro)
@@ -107,4 +107,20 @@
         </collision>
     </link>
+    <!-- End-effector (box of approximate size for now) -->
+    <link name="link6">
+        <visual>
+            <geometry>
+                <box size="0.12 0.12 0.26"/>
+            </geometry>
+            <origin xyz="0 0 0.13" rpy="0 0 0"/>
+            <material name="grey"/>
+        </visual>
+        <collision>
+            <geometry>
+                <box size="0.12 0.12 0.26"/>
+            </geometry>
+            <origin xyz="0 0 0.13" rpy="0 0 0"/>
+        </collision>
+    </link>
     <!-- Robot joints -->
     <joint name="world_to_linear_rail" type="fixed">
@@ -155,3 +171,10 @@
         <limit effort="24" velocity="3.5" lower="-3.14159" upper="3.14159"/>    <!-- Joint limits (effort, velocity, lower and upper angle limits in radians) -->
     </joint>
+    <joint name="joint6" type="revolute">
+        <parent link="link5"/>                                                  <!-- Parent link for joint6 -->
+        <child link="link6"/>                                                   <!-- Child link for joint6 -->
+        <origin xyz="-0.047 0 -0.055033" rpy="0 -1.57079 0"/>                   <!-- Origin of the joint -->
+        <axis xyz="0 0 1"/>                                                     <!-- Axis of rotation for the revolute joint (z-axis) -->
+        <limit effort="12" velocity="3.5" lower="-1.57079" upper="1.57079"/>    <!-- Joint limits (effort, velocity, lower and upper angle limits in radians) -->
+    </joint>
 </robot>

Commit message: feat(URDF): :rocket: Finish addition of gripper base link with fixed joint (joint 6) to URDF config
Finish addition of gripper base link and fixed joint 6 to URDF config

File: src/robot_description/urdf/robot.ros2_control.xacro (robot description, xacro)
@@ -49,11 +49,4 @@
                 <state_interface name="velocity"/>
             </joint>
-            <joint name="joint6">
-                <command_interface name="position"/>
-                <state_interface name="position">
-                    <param name="initial_value">0.0</param>
-                </state_interface>
-                <state_interface name="velocity"/>
-            </joint>
         </ros2_control>
     </xacro:macro>

File: src/robot_description/urdf/robot.xacro (robot description, xacro)
@@ -111,7 +111,7 @@
         <visual>
             <geometry>
-                <mesh filename="package://robot_description/meshes/Link 6 Visual.stl" scale="0.001 0.001 0.001"/>       <!-- Visual geometry for the end-effector link (STL file) -->
+                <mesh filename="package://robot_description/meshes/End Effector Geometry.stl" scale="0.001 0.001 0.001"/>       <!-- Visual geometry for the end-effector link (STL file) -->
             </geometry>
-            <origin xyz="0 0 0.13" rpy="0 0 0"/>
+            <origin xyz="0 0 0" rpy="0 0 0"/>
             <material name="grey"/>
         </visual>
@@ -120,5 +120,5 @@
                 <box size="0.12 0.12 0.26"/>                                                                            <!-- Collision geometry for the end-effector link (box shape) -->
             </geometry>
-            <origin xyz="0 0 0.13" rpy="0 0 0"/>
+            <origin xyz="0 0 0" rpy="0 0 0"/>
         </collision>
     </link>
@@ -171,10 +171,9 @@
         <limit effort="24" velocity="3.5" lower="-3.14159" upper="3.14159"/>    <!-- Joint limits (effort, velocity, lower and upper angle limits in radians) -->
     </joint>
-    <joint name="joint6" type="revolute">
+    <joint name="joint6" type="fixed">
         <parent link="link5"/>                                                  <!-- Parent link for joint6 -->
         <child link="link6"/>                                                   <!-- Child link for joint6 -->
         <origin xyz="-0.047 0 -0.055033" rpy="0 -1.57079 0"/>                   <!-- Origin of the joint -->
         <axis xyz="0 0 1"/>                                                     <!-- Axis of rotation for the revolute joint (z-axis) -->
-        <limit effort="12" velocity="3.5" lower="-1.57079" upper="1.57079"/>    <!-- Joint limits (effort, velocity, lower and upper angle limits in radians) -->
     </joint>
 </robot>

Commit message: feat(MoveIt): :construction: Start addition of gripper fins
Start addition of gripper fins

File: src/robot_description/urdf/robot.ros2_control.xacro (robot description, xacro)
@@ -49,4 +49,11 @@
                 <state_interface name="velocity"/>
             </joint>
+            <joint name="fin_joint1">
+                <command_interface name="position"/>
+                <state_interface name="position">
+                    <param name="initial_value">0.0</param>
+                </state_interface>
+                <state_interface name="velocity"/>
+            </joint>
         </ros2_control>
     </xacro:macro>

File: src/robot_description/urdf/robot.xacro (robot description, xacro)
@@ -118,5 +118,50 @@
         <collision>
             <geometry>
-                <box size="0.12 0.12 0.26"/>                                                                            <!-- Collision geometry for the end-effector link (box shape) -->
+                <mesh filename="package://robot_description/meshes/End Effector Geometry.stl" scale="0.001 0.001 0.001"/>    <!-- Collision geometry for the end-effector link (STL file) -->
+            </geometry>
+            <origin xyz="0 0 0" rpy="0 0 0"/>
+        </collision>
+    </link>
+    <link name="fin_link1">
+        <visual>
+            <geometry>
+                <mesh filename="package://robot_description/meshes/Gripper fin.stl" scale="0.001 0.001 0.001"/>       <!-- Visual geometry for the fin link 1 (STL file) -->
+            </geometry>
+            <origin xyz="0 0 0" rpy="0 0 0"/>
+            <material name="grey"/>
+        </visual>
+        <collision>
+            <geometry>
+                <mesh filename="package://robot_description/meshes/Gripper fin.stl" scale="0.001 0.001 0.001"/>    <!-- Collision geometry for the fin link 1 (STL file) -->
+            </geometry>
+            <origin xyz="0 0 0" rpy="0 0 0"/>
+        </collision>
+    </link>
+    <link name="fin_link2">
+        <visual>
+            <geometry>
+                <mesh filename="package://robot_description/meshes/Gripper fin.stl" scale="0.001 0.001 0.001"/>       <!-- Visual geometry for the fin link 1 (STL file) -->
+            </geometry>
+            <origin xyz="0 0 0" rpy="0 0 0"/>
+            <material name="grey"/>
+        </visual>
+        <collision>
+            <geometry>
+                <mesh filename="package://robot_description/meshes/Gripper fin.stl" scale="0.001 0.001 0.001"/>    <!-- Collision geometry for the fin link 1 (STL file) -->
+            </geometry>
+            <origin xyz="0 0 0" rpy="0 0 0"/>
+        </collision>
+    </link>
+    <link name="fin_link3">
+        <visual>
+            <geometry>
+                <mesh filename="package://robot_description/meshes/Gripper fin.stl" scale="0.001 0.001 0.001"/>       <!-- Visual geometry for the fin link 1 (STL file) -->
+            </geometry>
+            <origin xyz="0 0 0" rpy="0 0 0"/>
+            <material name="grey"/>
+        </visual>
+        <collision>
+            <geometry>
+                <mesh filename="package://robot_description/meshes/Gripper fin.stl" scale="0.001 0.001 0.001"/>    <!-- Collision geometry for the fin link 1 (STL file) -->
             </geometry>
             <origin xyz="0 0 0" rpy="0 0 0"/>
@@ -177,3 +222,26 @@
         <axis xyz="0 0 1"/>                                                     <!-- Axis of rotation for the revolute joint (z-axis) -->
     </joint>
+    <joint name="fin_joint1" type="revolute">
+        <parent link="link6"/>                                                  <!-- Parent link for fin_joint1 -->
+        <child link="fin_link1"/>                                               <!-- Child link for fin_joint1 -->
+        <origin xyz="0.049999999 0 0.1355" rpy="0 0 3.14159"/>                  <!-- Origin of the joint -->
+        <axis xyz="0 1 0"/>                                                     <!-- Axis of rotation for the revolute joint (y-axis) -->
+        <limit effort="10" velocity="1.0" lower="-1.0" upper="1.0"/>               <!-- Joint limits (effort, velocity, lower and upper angle limits in radians) -->
+    </joint>
+    <joint name="fin_joint2" type="revolute">
+        <parent link="link6"/>                                                  <!-- Parent link for fin_joint2 -->
+        <child link="fin_link2"/>                                               <!-- Child link for fin_joint2 -->
+        <origin xyz="-0.025 0.0433 0.1255" rpy="0 0 5.23599"/>                        <!-- Origin of the joint -->
+        <axis xyz="0 1 0"/>                                                     <!-- Axis of rotation for the revolute joint (y-axis) -->
+        <limit effort="10" velocity="1.0" lower="-1.0" upper="1.0"/>               <!-- Joint limits (effort, velocity, lower and upper angle limits in radians) -->
+        <mimic joint="fin_joint1" multiplier="1.0" offset="0.0"/>               <!-- Mimic joint definition to mirror the motion of fin_joint1 -->
+    </joint>
+    <joint name="fin_joint3" type="revolute">
+        <parent link="link6"/>                                                  <!-- Parent link for fin_joint3 -->
+        <child link="fin_link3"/>                                               <!-- Child link for fin_joint3 -->
+        <origin xyz="-0.025 -0.0433 0.1255" rpy="0 0 7.33039"/>                       <!-- Origin of the joint -->
+        <axis xyz="0 1 0"/>                                                     <!-- Axis of rotation for the revolute joint (y-axis) -->
+        <limit effort="10" velocity="1.0" lower="-1.0" upper="1.0"/>               <!-- Joint limits (effort, velocity, lower and upper angle limits in radians) -->
+        <mimic joint="fin_joint1" multiplier="1.0" offset="0.0"/>               <!-- Mimic joint definition to mirror the motion of fin_joint1 -->
+    </joint>
 </robot>

Commit message: build(URDF): :wrench: Update joint 6 to be revolute
Update joint 6 to be a revolute joint instead of fixed

File: src/robot_description/urdf/robot.ros2_control.xacro (robot description, xacro)
@@ -49,4 +49,11 @@
                 <state_interface name="velocity"/>
             </joint>
+            <joint name="joint6">
+                <command_interface name="position"/>
+                <state_interface name="position">
+                    <param name="initial_value">0.0</param>
+                </state_interface>
+                <state_interface name="velocity"/>
+            </joint>
             <joint name="fin_joint1">
                 <command_interface name="position"/>

File: src/robot_description/urdf/robot.xacro (robot description, xacro)
@@ -103,5 +103,5 @@
         <collision>
             <geometry>
-                <mesh filename="package://robot_description/meshes/Link 5 Collision.stl" scale="0.001 0.001 0.001"/>         <!-- Collision geometry for the link 5 (STL file) -->
+                <mesh filename="package://robot_description/meshes/Link 5 Visual.stl" scale="0.001 0.001 0.001"/>         <!-- Collision geometry for the link 5 (STL file) -->
             </geometry>
             <origin xyz="0 0 0" rpy="0 0 0"/>
@@ -214,11 +214,12 @@
         <origin xyz="-0.054 0 0.4645" rpy="0 1.57079 0"/>                       <!-- Origin of the joint -->
         <axis xyz="0 0 1"/>                                                     <!-- Axis of rotation for the revolute joint (z-axis) -->
-        <limit effort="24" velocity="3.5" lower="-3.14159" upper="3.14159"/>    <!-- Joint limits (effort, velocity, lower and upper angle limits in radians) -->
-    </joint>
-    <joint name="joint6" type="fixed">
+        <limit effort="24" velocity="3.5" lower="-5" upper="5"/>                <!-- Joint limits (effort, velocity, lower and upper angle limits in radians) -->
+    </joint>
+    <joint name="joint6" type="revolute">
         <parent link="link5"/>                                                  <!-- Parent link for joint6 -->
         <child link="link6"/>                                                   <!-- Child link for joint6 -->
         <origin xyz="-0.047 0 -0.055033" rpy="0 -1.57079 0"/>                   <!-- Origin of the joint -->
         <axis xyz="0 0 1"/>                                                     <!-- Axis of rotation for the revolute joint (z-axis) -->
+        <limit effort="24" velocity="3.5" lower="0" upper="2.0944"/>                <!-- Joint limits (effort, velocity, lower and upper angle limits in radians) -->
     </joint>
     <joint name="fin_joint1" type="revolute">
@@ -227,5 +228,5 @@
         <origin xyz="0.05052 0 0.1355" rpy="0 0 3.14159"/>                      <!-- Origin of the joint (hinge hole center at r=50.52mm, z=135.5mm) -->
         <axis xyz="0 1 0"/>                                                     <!-- Axis of rotation for the revolute joint (y-axis) -->
-        <limit effort="10" velocity="1.0" lower="-0.25" upper="0.175"/>            <!-- Joint limits (effort, velocity, lower and upper angle limits in radians) -->
+        <limit effort="10" velocity="1.0" lower="-0.25" upper="0.175"/>         <!-- Joint limits (effort, velocity, lower and upper angle limits in radians) -->
     </joint>
     <joint name="fin_joint2" type="revolute">
@@ -234,5 +235,5 @@
         <origin xyz="-0.02526 0.04375 0.1355" rpy="0 0 5.23599"/>               <!-- Origin of the joint (hinge hole center at r=50.52mm, 120°, z=135.5mm) -->
         <axis xyz="0 1 0"/>                                                     <!-- Axis of rotation for the revolute joint (y-axis) -->
-        <limit effort="10" velocity="1.0" lower="-0.25" upper="0.175"/>            <!-- Joint limits (effort, velocity, lower and upper angle limits in radians) -->
+        <limit effort="10" velocity="1.0" lower="-0.25" upper="0.175"/>         <!-- Joint limits (effort, velocity, lower and upper angle limits in radians) -->
         <mimic joint="fin_joint1" multiplier="1.0" offset="0.0"/>               <!-- Mimic joint definition to mirror the motion of fin_joint1 -->
     </joint>
@@ -242,5 +243,5 @@
         <origin xyz="-0.02526 -0.04375 0.1355" rpy="0 0 7.33039"/>              <!-- Origin of the joint (hinge hole center at r=50.52mm, 240°, z=135.5mm) -->
         <axis xyz="0 1 0"/>                                                     <!-- Axis of rotation for the revolute joint (y-axis) -->
-        <limit effort="10" velocity="1.0" lower="-0.25" upper="0.175"/>            <!-- Joint limits (effort, velocity, lower and upper angle limits in radians) -->
+        <limit effort="10" velocity="1.0" lower="-0.25" upper="0.175"/>         <!-- Joint limits (effort, velocity, lower and upper angle limits in radians) -->
         <mimic joint="fin_joint1" multiplier="1.0" offset="0.0"/>               <!-- Mimic joint definition to mirror the motion of fin_joint1 -->
     </joint>

Commit message: Update staged MoveIt and EPOS hardware configuration

File: src/robot_description/urdf/robot.ros2_control.xacro (robot description, xacro)
@@ -49,4 +49,11 @@
                 <state_interface name="velocity"/>
             </joint>
+            <joint name="joint6">
+                <command_interface name="position"/>
+                <state_interface name="position">
+                    <param name="initial_value">0.0</param>
+                </state_interface>
+                <state_interface name="velocity"/>
+            </joint>
             <joint name="fin_joint1">
                 <command_interface name="position"/>

File: src/robot_description/urdf/robot.xacro (robot description, xacro)
@@ -216,9 +216,10 @@
         <limit effort="24" velocity="3.5" lower="-3.14159" upper="3.14159"/>    <!-- Joint limits (effort, velocity, lower and upper angle limits in radians) -->
     </joint>
-    <joint name="joint6" type="fixed">
+    <joint name="joint6" type="revolute">
         <parent link="link5"/>                                                  <!-- Parent link for joint6 -->
         <child link="link6"/>                                                   <!-- Child link for joint6 -->
         <origin xyz="-0.047 0 -0.055033" rpy="0 -1.57079 0"/>                   <!-- Origin of the joint -->
         <axis xyz="0 0 1"/>                                                     <!-- Axis of rotation for the revolute joint (z-axis) -->
+        <limit effort="24" velocity="3.5" lower="-3.14159" upper="3.14159"/>
     </joint>
     <joint name="fin_joint1" type="revolute">
