Commit message: feat(URDF): :wrench: Add new named poses and rename old ones
Add new named poses ("vertical" and "bin") and renamed old poses ("home" to "crouch" and "zero" to "attention")

File: src/robot_description/urdf/robot.xacro (robot description, xacro)
@@ -142,5 +142,5 @@
         <origin xyz="0 0 0" rpy="0 0 0"/>                                       <!-- Origin of the joint -->
         <axis xyz="0 0 1"/>                                                     <!-- Axis of rotation for the revolute joint (z-axis) -->
-        <limit effort="37" velocity="0.4" lower="-3.14" upper="3.14"/>          <!-- Joint limits (effort, velocity, lower and upper angle limits in radians) -->
+        <limit effort="37" velocity="0.4" lower="-3.14159" upper="3.14159"/>          <!-- Joint limits (effort, velocity, lower and upper angle limits in radians) -->
     </joint>
     <joint name="joint2" type="revolute">

Commit message: style(URDF): :bulb: Update comments for links
Update comments for links in URDF

File: src/robot_description/urdf/robot.xacro (robot description, xacro)
@@ -6,14 +6,14 @@
         <visual>
             <geometry>
-                <box size="2.9464 0.445 0.1016"/>  <!-- Visual geometry for the linear rail (box shape) -->
+                <box size="2.9464 0.445 0.1016"/>                                                                        <!-- Visual geometry for the linear rail (box shape) -->
             </geometry>
-            <origin xyz="0 0 0" rpy="0 0 0"/>       <!-- Origin of the visual element (centered on the linear rail) -->
+            <origin xyz="0 0 0" rpy="0 0 0"/>
             <material name="grey"/>
         </visual>
         <collision>
             <geometry>
-                <box size="2.9464 0.445 0.1016"/>  <!-- Collision geometry for the linear rail (box shape) -->
+                <box size="2.9464 0.445 0.1016"/>                                                                        <!-- Collision geometry for the linear rail (box shape) -->
             </geometry>
-            <origin xyz="0 0 0" rpy="0 0 0"/>       <!-- Origin of the collision element (centered on the linear rail) -->
+            <origin xyz="0 0 0" rpy="0 0 0"/>
         </collision>
     </link>
@@ -21,7 +21,7 @@
         <visual>
             <geometry>
-                <mesh filename="package://robot_description/meshes/Base Link Visual.stl" scale="0.001 0.001 0.001"/>  <!-- Visual geometry for the base link (STL file) -->
+                <mesh filename="package://robot_description/meshes/Base Link Visual.stl" scale="0.001 0.001 0.001"/>     <!-- Visual geometry for the base link (STL file) -->
             </geometry>
-            <origin xyz="0 0 0" rpy="0 0 0"/>       <!-- Origin of the visual element (centered on the base link) -->
+            <origin xyz="0 0 0" rpy="0 0 0"/>
             <material name="grey"/>
         </visual>
@@ -30,5 +30,5 @@
                 <mesh filename="package://robot_description/meshes/Base Link Collision.stl" scale="0.001 0.001 0.001"/>  <!-- Collision geometry for the base link (STL file) -->
             </geometry>
-            <origin xyz="0 0 0" rpy="0 0 0"/>       <!-- Origin of the collision element (centered on the base link) -->
+            <origin xyz="0 0 0" rpy="0 0 0"/>
         </collision>
     </link>
@@ -36,5 +36,5 @@
         <visual>
             <geometry>
-                <mesh filename="package://robot_description/meshes/Link 1 Visual.stl" scale="0.001 0.001 0.001"/>  <!-- Visual geometry for the shoulder link (STL file) -->
+                <mesh filename="package://robot_description/meshes/Link 1 Visual.stl" scale="0.001 0.001 0.001"/>        <!-- Visual geometry for the link 1 (STL file) -->
             </geometry>
             <origin xyz="0 0 0" rpy="0 0 0"/>
@@ -43,5 +43,5 @@
         <collision>
             <geometry>
-                <mesh filename="package://robot_description/meshes/Link 1 Collision.stl" scale="0.001 0.001 0.001"/>  <!-- Collision geometry for the shoulder link (STL file) -->
+                <mesh filename="package://robot_description/meshes/Link 1 Collision.stl" scale="0.001 0.001 0.001"/>     <!-- Collision geometry for the link 1 (STL file) -->
             </geometry>
             <origin xyz="0 0 0" rpy="0 0 0"/>
@@ -51,5 +51,5 @@
         <visual>
             <geometry>
-                <mesh filename="package://robot_description/meshes/Link 2 Visual.stl" scale="0.001 0.001 0.001"/>  <!-- Visual geometry for the elbow link (STL file) -->
+                <mesh filename="package://robot_description/meshes/Link 2 Visual.stl" scale="0.001 0.001 0.001"/>        <!-- Visual geometry for the link 2 (STL file) -->
             </geometry>
             <origin xyz="0 0 0" rpy="0 0 0"/>
@@ -58,5 +58,5 @@
         <collision>
             <geometry>
-                <mesh filename="package://robot_description/meshes/Link 2 Collision.stl" scale="0.001 0.001 0.001"/>  <!-- Collision geometry for the elbow link (STL file) -->
+                <mesh filename="package://robot_description/meshes/Link 2 Collision.stl" scale="0.001 0.001 0.001"/>     <!-- Collision geometry for the link 2 (STL file) -->
             </geometry>
             <origin xyz="0 0 0" rpy="0 0 0"/>
@@ -66,5 +66,5 @@
         <visual>
             <geometry>
-                <mesh filename="package://robot_description/meshes/Link 3 Visual.stl" scale="0.001 0.001 0.001"/>  <!-- Visual geometry for the wrist link (STL file) -->
+                <mesh filename="package://robot_description/meshes/Link 3 Visual.stl" scale="0.001 0.001 0.001"/>        <!-- Visual geometry for the link 3 (STL file) -->
             </geometry>
             <origin xyz="0 0 0" rpy="0 0 0"/>
@@ -73,5 +73,5 @@
         <collision>
             <geometry>
-                <mesh filename="package://robot_description/meshes/Link 3 Collision.stl" scale="0.001 0.001 0.001"/>  <!-- Collision geometry for the wrist link (STL file) -->
+                <mesh filename="package://robot_description/meshes/Link 3 Collision.stl" scale="0.001 0.001 0.001"/>     <!-- Collision geometry for the link 3 (STL file) -->
             </geometry>
             <origin xyz="0 0 0" rpy="0 0 0"/>
@@ -81,5 +81,5 @@
         <visual>
             <geometry>
-                <mesh filename="package://robot_description/meshes/Link 4 Visual.stl" scale="0.001 0.001 0.001"/>  <!-- Visual geometry for the end-effector link (STL file) -->
+                <mesh filename="package://robot_description/meshes/Link 4 Visual.stl" scale="0.001 0.001 0.001"/>       <!-- Visual geometry for the link 4 (STL file) -->
             </geometry>
             <origin xyz="0 0 0" rpy="0 0 0"/>
@@ -88,5 +88,5 @@
         <collision>
             <geometry>
-                <mesh filename="package://robot_description/meshes/Link 4 Collision.stl" scale="0.001 0.001 0.001"/>  <!-- Collision geometry for the end-effector link (STL file) -->
+                <mesh filename="package://robot_description/meshes/Link 4 Collision.stl" scale="0.001 0.001 0.001"/>    <!-- Collision geometry for the link 4 (STL file) -->
             </geometry>
             <origin xyz="0 0 0" rpy="0 0 0"/>
@@ -96,5 +96,5 @@
         <visual>
             <geometry>
-                <mesh filename="package://robot_description/meshes/Link 5 Visual.stl" scale="0.001 0.001 0.001"/>  <!-- Visual geometry for the end-effector link (STL file) -->
+                <mesh filename="package://robot_description/meshes/Link 5 Visual.stl" scale="0.001 0.001 0.001"/>       <!-- Visual geometry for the link 5 (STL file) -->
             </geometry>
             <origin xyz="0 0 0" rpy="0 0 0"/>
@@ -103,14 +103,13 @@
         <collision>
             <geometry>
-                <mesh filename="package://robot_description/meshes/Link 5 Collision.stl" scale="0.001 0.001 0.001"/>  <!-- Collision geometry for the end-effector link (STL file) -->
+                <mesh filename="package://robot_description/meshes/Link 5 Collision.stl" scale="0.001 0.001 0.001"/>    <!-- Collision geometry for the link 5 (STL file) -->
             </geometry>
             <origin xyz="0 0 0" rpy="0 0 0"/>
         </collision>
     </link>
-    <!-- End-effector (box of approximate size for now) -->
     <link name="link6">
         <visual>
             <geometry>
-                <box size="0.12 0.12 0.26"/>
+                <mesh filename="package://robot_description/meshes/Link 6 Visual.stl" scale="0.001 0.001 0.001"/>       <!-- Visual geometry for the end-effector link (STL file) -->
             </geometry>
             <origin xyz="0 0 0.13" rpy="0 0 0"/>
@@ -119,5 +118,5 @@
         <collision>
             <geometry>
-                <box size="0.12 0.12 0.26"/>
+                <box size="0.12 0.12 0.26"/>                                                                            <!-- Collision geometry for the end-effector link (box shape) -->
             </geometry>
             <origin xyz="0 0 0.13" rpy="0 0 0"/>

Commit message: fix(URDF): 🔧Adjust linear rail link and joint for new 0 point

File: src/robot_description/urdf/robot.xacro (robot description, xacro)
@@ -6,5 +6,5 @@
         <visual>
             <geometry>
-                <box size="2.9464 0.445 0.1016"/>                                                                        <!-- Visual geometry for the linear rail (box shape) -->
+                <box size="2.97 0.45 0.082"/>                                                                        <!-- Visual geometry for the linear rail (box shape) -->
             </geometry>
             <origin xyz="0 0 0" rpy="0 0 0"/>
@@ -13,5 +13,5 @@
         <collision>
             <geometry>
-                <box size="2.9464 0.445 0.1016"/>                                                                        <!-- Collision geometry for the linear rail (box shape) -->
+                <box size="2.97 0.45 0.082"/>                                                                        <!-- Collision geometry for the linear rail (box shape) -->
             </geometry>
             <origin xyz="0 0 0" rpy="0 0 0"/>
@@ -134,5 +134,5 @@
         <origin xyz="0 0 0.0508" rpy="0 0 0"/>                                  <!-- Origin of the joint -->
         <axis xyz="1 0 0"/>                                                     <!-- Axis of translation for the prismatic joint (x-axis) -->
-        <limit effort="100" velocity="0.5" lower="-0.85" upper="0.85"/>         <!-- Joint limits (effort, velocity, lower and upper translation limits in meters) !! CHANGE LATER !! -->
+        <limit effort="100" velocity="0.5" lower="0" upper="0.1565"/>         <!-- Joint limits (effort, velocity, lower and upper translation limits in meters) !! CHANGE LATER !! -->
     </joint>
     <joint name="joint1" type="revolute">

Commit message: refactor(URDF): :wrench: Update linear rail link and joint config

File: src/robot_description/urdf/robot.xacro (robot description, xacro)
@@ -132,7 +132,7 @@
         <parent link="linear_rail_link"/>                                       <!-- Parent link for joint0 -->
         <child link="base_link"/>                                               <!-- Child link for joint0 -->
-        <origin xyz="0 0 0.0508" rpy="0 0 0"/>                                  <!-- Origin of the joint -->
+        <origin xyz="-0.7825 0 0.0508" rpy="0 0 0"/>                            <!-- Origin of the joint -->
         <axis xyz="1 0 0"/>                                                     <!-- Axis of translation for the prismatic joint (x-axis) -->
-        <limit effort="100" velocity="0.5" lower="0" upper="0.1565"/>         <!-- Joint limits (effort, velocity, lower and upper translation limits in meters) !! CHANGE LATER !! -->
+        <limit effort="100" velocity="0.5" lower="0" upper="1.565"/>            <!-- Joint limits are 0 = home end, 1.565 m = far end -->
     </joint>
     <joint name="joint1" type="revolute">
@@ -141,5 +141,5 @@
         <origin xyz="0 0 0" rpy="0 0 0"/>                                       <!-- Origin of the joint -->
         <axis xyz="0 0 1"/>                                                     <!-- Axis of rotation for the revolute joint (z-axis) -->
-        <limit effort="37" velocity="0.4" lower="-3.14159" upper="3.14159"/>          <!-- Joint limits (effort, velocity, lower and upper angle limits in radians) -->
+        <limit effort="37" velocity="0.4" lower="-3.14159" upper="3.14159"/>    <!-- Joint limits (effort, velocity, lower and upper angle limits in radians) -->
     </joint>
     <joint name="joint2" type="revolute">

Commit message: chore(URDF): :wrench: Fix fin mimic joint limits

File: src/robot_description/urdf/robot.xacro (robot description, xacro)
@@ -234,5 +234,5 @@
         <origin xyz="-0.02526 0.04375 0.1355" rpy="0 0 5.23599"/>               <!-- Origin of the joint (hinge hole center at r=50.52mm, 120°, z=135.5mm) -->
         <axis xyz="0 1 0"/>                                                     <!-- Axis of rotation for the revolute joint (y-axis) -->
-        <limit effort="10" velocity="1.0" lower="-1.0" upper="1.0"/>            <!-- Joint limits (effort, velocity, lower and upper angle limits in radians) -->
+        <limit effort="10" velocity="1.0" lower="-0.25" upper="0.175"/>            <!-- Joint limits (effort, velocity, lower and upper angle limits in radians) -->
         <mimic joint="fin_joint1" multiplier="1.0" offset="0.0"/>               <!-- Mimic joint definition to mirror the motion of fin_joint1 -->
     </joint>
@@ -242,5 +242,5 @@
         <origin xyz="-0.02526 -0.04375 0.1355" rpy="0 0 7.33039"/>              <!-- Origin of the joint (hinge hole center at r=50.52mm, 240°, z=135.5mm) -->
         <axis xyz="0 1 0"/>                                                     <!-- Axis of rotation for the revolute joint (y-axis) -->
-        <limit effort="10" velocity="1.0" lower="-1.0" upper="1.0"/>            <!-- Joint limits (effort, velocity, lower and upper angle limits in radians) -->
+        <limit effort="10" velocity="1.0" lower="-0.25" upper="0.175"/>            <!-- Joint limits (effort, velocity, lower and upper angle limits in radians) -->
         <mimic joint="fin_joint1" multiplier="1.0" offset="0.0"/>               <!-- Mimic joint definition to mirror the motion of fin_joint1 -->
     </joint>

Commit message: build(MoveIt): :wrench: Update configs for joint limits and controllers

File: src/robot_description/urdf/robot.xacro (robot description, xacro)
@@ -179,5 +179,5 @@
         <origin xyz="-0.7825 0 0.0508" rpy="0 0 0"/>                            <!-- Origin of the joint -->
         <axis xyz="1 0 0"/>                                                     <!-- Axis of translation for the prismatic joint (x-axis) -->
-        <limit effort="100" velocity="0.5" lower="0" upper="1.565"/>            <!-- Joint limits are 0 = home end, 1.565 m = far end -->
+        <limit effort="100" velocity="0.5" lower="0" upper="1.35"/>            <!-- Joint limits are 0 = home end, 1.565 m = far end -->
     </joint>
     <joint name="joint1" type="revolute">

Commit message: fix(URDF): :ambulance: Flip orientation of robot relative to world frame
Flip orientation of the robot relative to the world frame to be facing the +Y direction

File: src/robot_description/urdf/robot.xacro (robot description, xacro)
@@ -88,5 +88,5 @@
         <collision>
             <geometry>
-                <mesh filename="package://robot_description/meshes/Link 4 Collision.stl" scale="0.001 0.001 0.001"/>         <!-- Collision geometry for the link 4 (STL file) -->
+                <mesh filename="package://robot_description/meshes/Link 4 Visual.stl" scale="0.001 0.001 0.001"/>         <!-- Collision geometry for the link 4 (STL file) -->
             </geometry>
             <origin xyz="0 0 0" rpy="0 0 0"/>
@@ -172,5 +172,5 @@
         <parent link="world_frame"/>                                            <!-- Parent link for the fixed joint (world frame) -->
         <child link="linear_rail_link"/>                                        <!-- Child link for the fixed joint (linear rail) -->
-        <origin xyz="0 0 0" rpy="0 0 0"/>                                       <!-- Origin of the joint (position and orientation of the linear rail in the world frame) -->
+        <origin xyz="0 0 0" rpy="0 0 3.14159"/>                                 <!-- Origin of the joint (position and orientation of the linear rail in the world frame) -->
     </joint>
     <joint name="joint0" type="prismatic">
@@ -179,5 +179,5 @@
         <origin xyz="-0.7825 0 0.0508" rpy="0 0 0"/>                            <!-- Origin of the joint -->
         <axis xyz="1 0 0"/>                                                     <!-- Axis of translation for the prismatic joint (x-axis) -->
-        <limit effort="100" velocity="0.5" lower="0" upper="1.35"/>            <!-- Joint limits are 0 = home end, 1.565 m = far end -->
+        <limit effort="100" velocity="0.5" lower="0" upper="1.35"/>             <!-- Joint limits are 0 = home end, 1.565 m = far end -->
     </joint>
     <joint name="joint1" type="revolute">
@@ -200,5 +200,5 @@
         <origin xyz="-0.017125 0 0.663309" rpy="0 -1.57079 3.14195"/>           <!-- Origin of the joint -->
         <axis xyz="0 0 1"/>                                                     <!-- Axis of rotation for the revolute joint (z-axis) -->
-        <limit effort="77" velocity="3.65" lower="-4.5" upper="1.4"/>           <!-- Joint limits (effort, velocity, lower and upper angle limits in radians) -->
+        <limit effort="77" velocity="3.65" lower="-4.5" upper="1.5"/>           <!-- Joint limits (effort, velocity, lower and upper angle limits in radians) -->
     </joint>
     <joint name="joint4" type="revolute">
@@ -221,5 +221,5 @@
         <origin xyz="-0.047 0 -0.055033" rpy="0 -1.57079 0"/>                   <!-- Origin of the joint -->
         <axis xyz="0 0 1"/>                                                     <!-- Axis of rotation for the revolute joint (z-axis) -->
-        <limit effort="24" velocity="3.5" lower="0" upper="2.0944"/>                <!-- Joint limits (effort, velocity, lower and upper angle limits in radians) -->
+        <limit effort="24" velocity="3.5" lower="0" upper="2.0944"/>            S<!-- Joint limits (effort, velocity, lower and upper angle limits in radians) -->
     </joint>
     <joint name="fin_joint1" type="revolute">

Commit message: fix(URDF): :ambulance: *Actually* fix orientation of robot

File: src/robot_description/urdf/robot.xacro (robot description, xacro)
@@ -172,10 +172,10 @@
         <parent link="world_frame"/>                                            <!-- Parent link for the fixed joint (world frame) -->
         <child link="linear_rail_link"/>                                        <!-- Child link for the fixed joint (linear rail) -->
-        <origin xyz="0 0 0" rpy="0 0 3.14159"/>                                 <!-- Origin of the joint (position and orientation of the linear rail in the world frame) -->
+        <origin xyz="0 0 0" rpy="0 0 0"/>                                 <!-- Origin of the joint (position and orientation of the linear rail in the world frame) -->
     </joint>
     <joint name="joint0" type="prismatic">
         <parent link="linear_rail_link"/>                                       <!-- Parent link for joint0 -->
         <child link="base_link"/>                                               <!-- Child link for joint0 -->
-        <origin xyz="-0.7825 0 0.0508" rpy="0 0 0"/>                            <!-- Origin of the joint -->
+        <origin xyz="0.7825 0 0.0508" rpy="0 0 3.14159"/>                            <!-- Origin of the joint -->
         <axis xyz="1 0 0"/>                                                     <!-- Axis of translation for the prismatic joint (x-axis) -->
         <limit effort="100" velocity="0.5" lower="0" upper="1.35"/>             <!-- Joint limits are 0 = home end, 1.565 m = far end -->
